Commit message: igvcurdf.urdf.xacro

File: urdf/igvcurdf.urdf.xacro (robot description, xacro)
@@ -1,4 +1,31 @@
 <?xml version="1.0"?>
 <robot xmlns:xacro="http://www.ros.org/wiki/xacro" name="diffbot">
+<xacro:macro name="inertial_sphere" params="mass radius *origin">
+        <inertial>
+            <xacro:insert_block name="origin"/>
+            <mass value="${mass}" />
+            <inertia ixx="${(2/5) * mass * (radius*radius)}" ixy="0.0" ixz="0.0"
+                    iyy="${(2/5) * mass * (radius*radius)}" iyz="0.0"
+                    izz="${(2/5) * mass * (radius*radius)}" />
+        </inertial>
+    </xacro:macro>
+    <xacro:macro name="inertial_box" params="mass x y z *origin">
+        <inertial>
+            <xacro:insert_block name="origin"/>
+            <mass value="${mass}" />
+            <inertia ixx="${(1/12) * mass * (y*y+z*z)}" ixy="0.0" ixz="0.0"
+                    iyy="${(1/12) * mass * (x*x+z*z)}" iyz="0.0"
+                    izz="${(1/12) * mass * (x*x+y*y)}" />
+        </inertial>
+    </xacro:macro>
+    <xacro:macro name="inertial_cylinder" params="mass length radius *origin">
+        <inertial>
+            <xacro:insert_block name="origin"/>
+            <mass value="${mass}" />
+            <inertia ixx="${(1/12) * mass * (3*radius*radius + length*length)}" ixy="0.0" ixz="0.0"
+                    iyy="${(1/12) * mass * (3*radius*radius + length*length)}" iyz="0.0"
+                    izz="${(1/2) * mass * (radius*radius)}" />
+        </inertial>
+    </xacro:macro>
 <!--colours-->
 <material name="red">
@@ -33,7 +60,7 @@
         </geometry>
     </collision>
-    <inertial>
-        <mass value="0.5"/>
-    </inertial>
+     <xacro:inertial_box mass="0.5" x="0.3" y="0.3" z="0.15">
+            <origin xyz="0.15 0 0.075" rpy="0 0 0"/>
+        </xacro:inertial_box>
 </link>
 <!-- wheels-->
@@ -56,7 +83,7 @@
         </geometry>
     </collision>
-   <inertial>
-        <mass value="0.05"/>
-    </inertial>
+   <xacro:inertial_cylinder mass="0.1" length="0.05" radius="0.06">
+            <origin xyz="0 0 0" rpy="0 0 0"/>
+        </xacro:inertial_cylinder>
 </link>
 <joint name="right_wheel_joint" type="continuous">
@@ -78,7 +105,7 @@
         </geometry>
     </collision>
-   <inertial>
-        <mass value="0.05"/>
-    </inertial>
+   <xacro:inertial_cylinder mass="0.1" length="0.05" radius="0.06">
+            <origin xyz="0 0 0" rpy="0 0 0"/>
+        </xacro:inertial_cylinder>
 </link>
 <!--caster wheel-->
@@ -100,7 +127,7 @@
         </geometry>
     </collision>
-    <inertial>
-        <mass value="0.02"/>
-    </inertial>
+    <xacro:inertial_sphere mass="0.1" radius="0.025">
+            <origin xyz="0 0 0" rpy="0 0 0"/>
+        </xacro:inertial_sphere>
 </link>
 </robot>

Commit message: igvcurdf.urdf.xacro

File: urdf/igvcurdf.urdf.xacro (robot description, xacro)
@@ -1,4 +1,5 @@
 <?xml version="1.0"?>
 <robot xmlns:xacro="http://www.ros.org/wiki/xacro" name="diffbot">
+<xacro:include filename="gazebo_control.xacro"/>
 <xacro:macro name="inertial_sphere" params="mass radius *origin">
         <inertial>
@@ -63,4 +64,7 @@
             <origin xyz="0.15 0 0.075" rpy="0 0 0"/>
         </xacro:inertial_box>
+        <gazebo reference="chassis">
+            <material>Gazebo/red</material>
+        </gazebo>
 </link>
 <!-- wheels-->
@@ -86,4 +90,7 @@
             <origin xyz="0 0 0" rpy="0 0 0"/>
         </xacro:inertial_cylinder>
+        <gazebo reference="left_wheel">
+            <material>Gazebo/black</material>
+        </gazebo>
 </link>
 <joint name="right_wheel_joint" type="continuous">
@@ -108,4 +115,7 @@
             <origin xyz="0 0 0" rpy="0 0 0"/>
         </xacro:inertial_cylinder>
+        <gazebo reference="right_wheel">
+            <material>Gazebo/black</material>
+        </gazebo>
 </link>
 <!--caster wheel-->
@@ -118,5 +128,5 @@
     <visual>
         <geometry>
-            <sphere radius="0.025"/>
+            <sphere radius="0.06"/>
         </geometry>
         <material name="black"/>
@@ -124,10 +134,13 @@
     <collision>
         <geometry>
-            <sphere radius="0.025"/>
+            <sphere radius="0.06"/>
         </geometry>
     </collision>
-    <xacro:inertial_sphere mass="0.1" radius="0.025">
+    <xacro:inertial_sphere mass="0.1" radius="0.06">
             <origin xyz="0 0 0" rpy="0 0 0"/>
         </xacro:inertial_sphere>
+        <gazebo reference="caster">
+            <material>Gazebo/black</material>
+        </gazebo>
 </link>
 </robot>

Commit message: igvcurdf.urdf.xacro

File: urdf/igvcurdf.urdf.xacro (robot description, xacro)
@@ -72,6 +72,6 @@
     <parent link="chassis"/>
     <child link="left_wheel"/>
-    <origin xyz="0.05 0.175 0" rpy="-${pi/2} 0 0"/>
-    <axis  xyz="0 0 1"/>
+    <origin xyz="0.05 0.175 0" rpy="${pi/2} 0 0"/>
+    <axis  xyz="0 0 -1"/>
 </joint>
 <link name="left_wheel">
@@ -98,5 +98,5 @@
     <child link="right_wheel"/>
     <origin xyz="0.05 -0.175 0" rpy="${pi/2} 0 0"/>
-    <axis xyz="0 0 1"/>
+    <axis xyz="0 0 -1"/>
 </joint>
 <link name="right_wheel">

Commit message: igvcurdf.urdf.xacro

File: urdf/igvcurdf.urdf.xacro (robot description, xacro)
@@ -64,8 +64,8 @@
             <origin xyz="0.15 0 0.075" rpy="0 0 0"/>
         </xacro:inertial_box>
-        <gazebo reference="chassis">
+</link>
+<gazebo reference="chassis">
             <material>Gazebo/red</material>
         </gazebo>
-</link>
 <!-- wheels-->
 <joint name="left_wheel_joint" type="continuous">
@@ -90,8 +90,8 @@
             <origin xyz="0 0 0" rpy="0 0 0"/>
         </xacro:inertial_cylinder>
-        <gazebo reference="left_wheel">
+</link>
+<gazebo reference="left_wheel">
             <material>Gazebo/black</material>
         </gazebo>
-</link>
 <joint name="right_wheel_joint" type="continuous">
     <parent link="chassis"/>
@@ -115,8 +115,8 @@
             <origin xyz="0 0 0" rpy="0 0 0"/>
         </xacro:inertial_cylinder>
-        <gazebo reference="right_wheel">
+</link>
+<gazebo reference="right_wheel">
             <material>Gazebo/black</material>
         </gazebo>
-</link>
 <!--caster wheel-->
 <joint name="caster_joint" type="fixed">
@@ -140,7 +140,9 @@
             <origin xyz="0 0 0" rpy="0 0 0"/>
         </xacro:inertial_sphere>
-        <gazebo reference="caster">
+</link>
+<gazebo reference="caster">
             <material>Gazebo/black</material>
+            <mu1 value="0.0001"/>
+            <mu2 value="0.0001"/>
         </gazebo>
-</link>
 </robot>

Commit message: Update igvcurdf.urdf.xacro

File: urdf/igvcurdf.urdf.xacro (robot description, xacro)
@@ -43,4 +43,11 @@
 <!-- chassis-->
 <link name="base_link">
+</link>
+<joint name="base_footprint_joint" type="fixed">
+    <parent link="base_link"/>
+    <child link="base_footprint"/>
+    <origin xyz="0 0 0" rpy="0 0 0"/>
+</joint>
+<link name="base_footprint">
 </link>
 <joint name="chassis_joint" type="fixed">
